File: preamp2.sch (KiCad schematic (older format))
At the start: 56 parts, among them J1 Signal in, J2 AC in, J3 Signal out, J4 uC, U1 OPA2134, U2 PGA2311, U3 LM317_3PinPackage, U4 LM337_SOT223, U5 LM7805_TO220

Commit message: Decreased resistor value to increase possible current
Parts:
- R5, R6: value 10 -> 4.7
Changed lines of the file:
@@
 P 1700 5500
 F 0 "R5" V 1907 5500 50  0000 C CNN
-F 1 "10" V 1816 5500 50  0000 C CNN
+F 1 "4.7" V 1816 5500 50  0000 C CNN
 F 2 "Resistors_SMD:R_1218_HandSoldering" V 1630 5500 50  0001 C CNN
 F 3 "" H 1700 5500 50  0001 C CNN
@@
 P 1700 6700
 F 0 "R6" V 1907 6700 50  0000 C CNN
-F 1 "10" V 1816 6700 50  0000 C CNN
+F 1 "4.7" V 1816 6700 50  0000 C CNN
 F 2 "Resistors_SMD:R_1218_HandSoldering" V 1630 6700 50  0001 C CNN
 F 3 "" H 1700 6700 50  0001 C CNN

Commit message: Increased pin header size
Parts:
- J4: footprint Pin_Headers:Pin_Header_Straight_2x04_Pitch1.00mm -> Pin_Headers:Pin_Header_Straight_2x04_Pitch2.54mm
Changed lines of the file:
@@
 F 0 "J4" H 10100 1565 50  0000 C CNN
 F 1 "uC" H 10100 1474 50  0000 C CNN
-F 2 "Pin_Headers:Pin_Header_Straight_2x04_Pitch1.00mm" H 10100 0   50  0001 C CNN
+F 2 "Pin_Headers:Pin_Header_Straight_2x04_Pitch2.54mm" H 10100 0   50  0001 C CNN
 F 3 "" H 10100 0   50  0001 C CNN
 	1    10100 1200
