File: preamp2.kicad_pcb (KiCad board)
At the start: 2 copper layers, 60 parts, among them J1 Signal in, J2 AC in, J3 Signal out, J4 uC, U1 OPA2134, U2 PGA2311, U3 LM317_3PinPackage, U4 LM337_SOT223, U5 LM7805_TO220

Commit message: Increased pin header size
Parts:
- J4: footprint Pin_Headers:Pin_Header_Straight_2x04_Pitch1.00mm -> Pin_Headers:Pin_Header_Straight_2x04_Pitch2.54mm
- R5, R6: value 10 -> 4.7
- moved J4 2.81 mm to (120.7, 127.5)
Connections:
- REF** pad 1: (no net) -> GNDA
Routing:
- net VD: track 132.9 -> 125.2 mm
- net Mute: track 15.2 -> 17.9 mm
- net SDO: track 14.4 -> 16.3 mm
- net Zcen: track 16.9 -> 18.6 mm
- net GNDA: track 38.6 -> 37.6 mm
- net SDI: track 14.2 -> 13.2 mm
- net CLK: track 13.7 -> 14.5 mm
Other:
- board outline added: 84.8 x 54.4 mm

Commit message: Added some silk screen annotations
Parts:
- 4.7 Ω: renamed from R5
- 4.7 Ω: renamed from R6
- renumbered U3 to LM317, U4 to LM337, U5 to LM7805, U1 to OPA2134, U2 to PGA2311
Other:
- board text added: "6–9 VAC"
- board text added: "CLK"
- board text added: "CS"
- board text added: "GND"
- board text added: "Mute"
- board text added: "SDI"
- board text added: "SDO"
- board text added: "VD"
- board text added: "Va in"
- board text added: "Va out"
- board text added: "Vb in"
- board text added: "Vb out"
- board text added: "ZC"
Changed lines of the file:
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@@
   (general
     (thickness 1.6)
-    (drawings 5)
+    (drawings 20)
     (tracks 300)
     (zones 0)
@@
     (tags "SOIC 1.27")
     (attr smd)
-    (fp_text reference U1 (at -1.778 -3.5) (layer F.SilkS)
-      (effects (font (size 1 1) (thickness 0.15)))
+    (fp_text reference OPA2134 (at -1.524 -3.048) (layer F.SilkS)
+      (effects (font (size 0.6 0.6) (thickness 0.15)))
     )
     (fp_text value OPA2134 (at 0 3.5) (layer F.Fab)
@@
     (tags "SOIC 1.27")
     (attr smd)
-    (fp_text reference U2 (at 0 -6.25) (layer F.SilkS)
-      (effects (font (size 1 1) (thickness 0.15)))
+    (fp_text reference PGA2311 (at 0 -6.25) (layer F.SilkS)
+      (effects (font (size 0.6 0.6) (thickness 0.15)))
     )
     (fp_text value PGA2311 (at 0 6.25) (layer F.Fab)
@@
     (tags "CMS SOT")
     (attr smd)
-    (fp_text reference U3 (at 0 4.5 270) (layer B.SilkS)
+    (fp_text reference LM317 (at 0 -4.572 270) (layer B.SilkS)
       (effects (font (size 1 1) (thickness 0.15)) (justify mirror))
     )
@@
     (tags "CMS SOT")
     (attr smd)
-    (fp_text reference U4 (at 0 4.5 90) (layer B.SilkS)
+    (fp_text reference LM337 (at 0 4.5 90) (layer B.SilkS)
       (effects (font (size 1 1) (thickness 0.15)) (justify mirror))
     )
@@
     (descr "TO-220, Vertical, RM 2.54mm")
     (tags "TO-220 Vertical RM 2.54mm")
-    (fp_text reference U5 (at 2.54 -3.62 90) (layer F.SilkS)
+    (fp_text reference LM7805 (at 2.54 -3.62 90) (layer F.SilkS)
       (effects (font (size 1 1) (thickness 0.15)))
     )
@@
     (tags "resistor 1218")
     (attr smd)
-    (fp_text reference R5 (at 0 -3.5) (layer F.SilkS)
+    (fp_text reference "4.7 Ω" (at 0 -3.5) (layer F.SilkS)
       (effects (font (size 1 1) (thickness 0.15)))
     )
@@
     (tags "resistor 1218")
     (attr smd)
-    (fp_text reference R6 (at 0 -3.5) (layer F.SilkS)
+    (fp_text reference "4.7 Ω" (at -0.254 3.81) (layer F.SilkS)
       (effects (font (size 1 1) (thickness 0.15)))
     )
@@
     )
   )
+  (gr_text "Vb out" (at 166.37 99.822 90) (layer F.SilkS)
+    (effects (font (size 0.7 0.7) (thickness 0.175)))
+  )
+  (gr_text GND (at 166.37 104.902 90) (layer F.SilkS)
+    (effects (font (size 0.7 0.7) (thickness 0.175)))
+  )
+  (gr_text "Va out" (at 166.37 109.728 90) (layer F.SilkS)
+    (effects (font (size 0.7 0.7) (thickness 0.175)))
+  )
+  (gr_text "Vb in" (at 145.542 81.28 180) (layer F.SilkS)
+    (effects (font (size 0.7 0.7) (thickness 0.175)))
+  )
+  (gr_text "Va in" (at 135.636 81.28 180) (layer F.SilkS)
+    (effects (font (size 0.7 0.7) (thickness 0.175)))
+  )
+  (gr_text GND (at 140.462 81.28 180) (layer F.SilkS)
+    (effects (font (size 0.7 0.7) (thickness 0.175)))
+  )
+  (gr_text "6–9 VAC" (at 104.394 131.572) (layer F.SilkS)
+    (effects (font (size 0.7 0.7) (thickness 0.175)))
+  )
+  (gr_text Mute (at 113.03 132.08) (layer F.SilkS)
+    (effects (font (size 0.7 0.7) (thickness 0.175)))
+  )
+  (gr_text SDO (at 115.57 132.08) (layer F.SilkS)
+    (effects (font (size 0.7 0.7) (thickness 0.175)))
+  )
+  (gr_text CLK (at 118.11 132.08) (layer F.SilkS)
+    (effects (font (size 0.7 0.7) (thickness 0.175)))
+  )
+  (gr_text GND (at 120.65 132.08) (layer F.SilkS)
+    (effects (font (size 0.7 0.7) (thickness 0.175)))
+  )
+  (gr_text ZC (at 113.03 125.476) (layer F.SilkS)
+    (effects (font (size 0.7 0.7) (thickness 0.175)))
+  )
+  (gr_text CS (at 115.57 125.476) (layer F.SilkS)
+    (effects (font (size 0.7 0.7) (thickness 0.175)))
+  )
+  (gr_text SDI (at 118.11 125.476) (layer F.SilkS)
+    (effects (font (size 0.7 0.7) (thickness 0.175)))
+  )
+  (gr_text VD (at 120.65 125.476) (layer F.SilkS)
+    (effects (font (size 0.7 0.7) (thickness 0.175)))
+  )
   (gr_line (start 168.148 132.588) (end 168.148 78.232) (layer Edge.Cuts) (width 0.001))
